File: Matériel/1.2/ProgrammateurFilPilote_1.2.brd (EAGLE design)
At the start: 85.5 x 66.8 mm, 78 parts, among them IC2 MCP23017, J2 GROVE-I2C, P1 PADSMALL, P2 PADSMALL, SW1 HLS8L-DC5V-S-C, T1 2N2222

Commit message: Révision 1.2c
Parts:
- OP1, OP10, OP11, OP12, OP13, OP14, OP2, OP3, OP4, OP5, OP6, OP7, OP8, OP9: device TLP168J:MFSOP-4 -> TLP168J:MFSOP-4-HANDSOLDER
- moved LED 10.2 mm to (69.3, 36.3), turned to 90 degrees
- moved L 7.75 mm to (67.3, 36.2), turned to 270 degrees
- moved P2 5.76 mm to (62.2, 28.7)
- moved R21 5.12 mm to (64.5, 31.6)
- moved LOGO1 2.82 mm to (70.0, 29.7)
- moved LOGO2 2.32 mm to (70.0, 30.2)
- moved RX-433MHZ 1.37 mm to (64.6, 60.7)
- moved J2 0.63 mm to (70.4, 59.7)
Connections:
- net +3V3: now also EXTENSION.5; no longer EXTENSION.4
- net GND: now also EXTENSION.4; no longer EXTENSION.5
Routing:
- net PHASE: track 111.3 -> 131.6 mm
- net +3V3: track 163.2 -> 170.0 mm
- net N$6: track 3.92 -> 9.75 mm
- net SDA: track 130.1 -> 128.3 mm
- net LED: track 13.8 -> 12.5 mm
- net +5V: track 113.3 -> 114.3 mm
Other:
- board text added: "Programmateur Fil Pilote (v1.2c - 01/2015)"
- board text removed: "Programmateur Fil Pilote (v1.2b - 01/2015)"
