File: Matériel/1.3/ProgrammateurFilPilote_1.3.sch (EAGLE design)
At the start: 84 parts, among them IC1 MCP23017, J2 GROVE-I2C, P1 PADSMALL, P2 PADSMALL, SW1 HLS8L-DC5V-S-C, T1 2N3904, T2 BSS138

Commit message: Ajustements Finaux
Résistances 390 Ohm pour nouveaux optos Sharp
Commandes Opto/led via MCP par la masse
Ajustement des borniers pour boitier rail DIN
Parts:
- removed EXTENSION: (no value), con-ptr500:AK500/5
- removed F1: 1,25A temporisé, fuse:TE5
- added JP1: (no value), SparkFun-Connectors:M02PTH
- added OPTO: JUMPER-PAD-3-2OF3_NC_BY_TRACE_LARGE, SparkFun-Passives:JUMPER-PAD-3-2OF3_NC_BY_TRACE_LARGE
- added X1: (no value), con-ptr500:AK500/3
- LED: value LED3MMNOSILK -> LED3MM; device _c2h:LED3MMNOSILK -> _c2h:LED3MM
- R10, R11, R12, R13, R14, R15, R16, R21, R3, R4, R5, R6, R7, R8, R9: value 470 -> 390
- renumbered SJ1 to RGB
Connections:
- removed net PHASE-SECTEUR: 230V-1.KL, F1.1
- new net N$18: OP9.3, R11.2
- net +3V3: now also OPTO.1, X1-3.KL; no longer EXTENSION-5.KL
- net +5V: now also OPTO.3, X1-1.KL; no longer EXTENSION-3.KL
- net GND: now also X1-2.KL; no longer EXTENSION-4.KL, LED.MINUS, OP1.3, OP10.3, OP11.3, OP12.3, OP13.3, OP14.3, OP2.3, OP3.3, OP4.3, OP5.3, OP6.3, OP7.3, OP8.3, OP9.3
- net LED: now also R21.1; no longer R21.2
- net N$10: now also OP4.3; no longer OP4.1
- net N$11: now also OP5.3; no longer OP5.1
- net N$12: now also OP6.3; no longer OP6.1
- net N$13: now also OP7.3; no longer OP7.1
- net N$14: now also OP8.3; no longer OP8.1
- net N$19: now also LED.PLUS, OP1.1, OP10.1, OP11.1, OP12.1, OP13.1, OP14.1, OP2.1, OP3.1, OP4.1, OP5.1, OP6.1, OP7.1, OP8.1, OPTO.2; no longer R11.2
- net N$32: now also OP10.3; no longer OP10.1
- net N$34: now also OP14.3; no longer OP14.1
- net N$47: now also OP11.3; no longer OP11.1
- net N$48: now also OP12.3; no longer OP12.1
- net N$6: now also LED.MINUS, R21.2; no longer LED.PLUS, R21.1
- net N$7: now also OP1.3; no longer OP1.1
- net N$8: now also OP2.3; no longer OP2.1
- net N$9: now also OP3.3; no longer OP3.1
- net PHASE: now also 230V-1.KL; no longer F1.2
- net S$5: now also OP13.3; no longer OP13.1
- net SCL: now also JP1.2; no longer EXTENSION-1.KL
- net SDA: now also JP1.1; no longer EXTENSION-2.KL
Other:
- moved on the sheet: OP1, OP10, OP11, OP12, OP13, OP14, OP2, OP3, OP4, OP5, OP6, OP7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
